File: Melty/Melty.kicad_pcb (KiCad board)
At the start: 6 copper layers, 54.3 x 22 mm, 38 parts, among them J1 ESC signal, J2 ESC Power, J3 ESC Power, J4 Power In, J5 Switch, Q1 BSS138, Q2 BSS138, Q3 BSS138, U1 XIAO-ESP32-C3-DIP, U2 H3LIS331DLTR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

Commit message: PCB Ordered
Parts:
- added G***: LOGO, LOGO, B.Cu at (169.0, 56.3)
Routing:
- net +5V: vias 21 -> 22
Other:
- board text added: "Ethan Cao Melty V1"

Commit message: crsf reading
Changed lines of the file:
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@@
 		(fp_arc
 			(start 8.883636 8.56)
-			(mid 8.325678 9.907043)
+			(mid 8.325677 9.90704)
 			(end 6.978636 10.465)
 			(stroke
@@
 		(fp_arc
 			(start 6.978636 -10.49)
-			(mid 8.325674 -9.932037)
+			(mid 8.325671 -9.932036)
 			(end 8.883636 -8.585)
 			(stroke
@@
 		(fp_arc
 			(start 3.997636 -12)
-			(mid 4.351188 -11.853554)
+			(mid 4.351186 -11.853551)
 			(end 4.497636 -11.5)
 			(stroke

Commit message: FASTLED BADDDD
Parts:
- R7: value 50k -> 51k
Changed lines of the file:
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@@
 			)
 		)
-		(property "Value" "50k"
+		(property "Value" "51k"
 			(at 0 1.43 0)
 			(layer "F.Fab")
@@
 		(fp_arc
 			(start 8.883636 8.56)
-			(mid 8.325677 9.90704)
+			(mid 8.325678 9.907043)
 			(end 6.978636 10.465)
 			(stroke
@@
 		(fp_arc
 			(start 6.978636 -10.49)
-			(mid 8.325671 -9.932036)
+			(mid 8.325674 -9.932037)
 			(end 8.883636 -8.585)
 			(stroke
@@
 		(fp_arc
 			(start 3.997636 -12)
-			(mid 4.351186 -11.853551)
+			(mid 4.351166 -11.853541)
 			(end 4.497636 -11.5)
 			(stroke
@@
 		(sheetname "Root")
 		(sheetfile "Melty.kicad_sch")
-		(attr smd)
+		(attr smd dnp)
 		(fp_line
 			(start -0.65 1.56)
@@
 		(sheetname "Root")
 		(sheetfile "Melty.kicad_sch")
-		(attr smd)
+		(attr smd dnp)
 		(fp_line
 			(start 0.146267 0.51)
@@
 		(sheetname "Root")
 		(sheetfile "Melty.kicad_sch")
-		(attr smd)
+		(attr smd dnp)
 		(fp_line
 			(start 0.146267 0.51)
@@
 		(sheetname "Root")
 		(sheetfile "Melty.kicad_sch")
-		(attr smd)
+		(attr smd dnp)
 		(fp_line
 			(start 0.65 -1.56)
@@
 		(sheetname "Root")
 		(sheetfile "Melty.kicad_sch")
-		(attr smd)
+		(attr smd dnp)
 		(fp_line
 			(start 0.146267 -0.51)
@@
 		(sheetname "Root")
 		(sheetfile "Melty.kicad_sch")
-		(attr smd)
+		(attr smd dnp)
 		(fp_line
 			(start 0.146267 0.51)
